File: Proyecto/proyecto.kicad_pcb (KiCad board)
At the start: 2 copper layers, 75.2 x 72.9 mm, 17 parts, among them U1 PIC18F2550, U2 LM1117-TO, U3 RN42XV, U4 PICKIT3, U5 POLOLUV1, X1 20MHz

Commit message: Placa
Parts:
- moved U5 11.8 mm to (179.7, 95.9)
- moved U3 7.92 mm to (189.1, 121.8), turned to 0 degrees
- moved C2 1.45 mm to (166.1, 106.8)
- turned D1 to 0 degrees
- turned D2 to 0 degrees
Connections:
- D1 pad 1: N-0000045 -> N-0000047
- D1 pad 2: N-0000047 -> N-0000045
- D2 pad 1: N-0000046 -> N-0000048
- D2 pad 2: N-0000048 -> N-0000046
Routing:
- net /RX: track 11.6 -> 39.3 mm
- net /TX: track 11.4 -> 37.9 mm
- net /SDA: track 33.1 -> 22.4 mm
- net /SCL: track 33.1 -> 22.4 mm
- net /3V3: track 155.4 -> 158.4 mm
